File: hardware/WaterLevelMonitor_v1.brd (EAGLE design)
At the start: 98.7 x 49.5 mm, 42 parts, among them J1 D24V5F5, J2 AVR_SPI_PRG_6PTH, J5 D24V5F5, J6 D24V5F5, J7 RJ45, Q1 NDP6020P, Q4 2N3904, U1 ATMEGA328P_PDIP

Commit message: Add files via upload
Parts:
- added D2: (no value), adafruit:DO-1N4148
- added J8: (no value), SparkFun-Connectors:1X04
- added J9: (no value), SparkFun-Connectors:1X03
- D1: value (none) -> 1N5819-B; device adafruit:DO-1N4148 -> diode:DO41-7.6
- moved J3 48.6 mm to (59.7, 44.5), turned to 270 degrees
- moved D1 37.9 mm to (-10.2, -90.2)
- moved R3 20.1 mm to (68.6, 24.1), turned to 90 degrees
Connections:
- removed net BATSW: R3.2
- new net N$12: J3.7, U1.6
- new net N$13: D2.C, J8.2
- new net N$15: D2.A, U1.2
- new net N$16: J3.9, U1.5
- new net N$17: J3.10, U1.4
- new net N$18: J8.1, J9.2
- new net N$19: R3.2, U1.28
- new net N$7: J8.3, U1.3
- net GND: now also J3.2, J8.4
- net N$4: now also J3.12
- net N$6: now also U1.23
- net VCC: now also J9.1
- net VCEL: now also J3.1
- net VSEN: now also J9.3
Routing:
- net VBAT: track 73.0 -> 0.00 mm
- net N$3: track 23.2 -> 0.00 mm
- net N$1: track 14.5 -> 0.00 mm
- net N$5: track 7.62 -> 0.00 mm
- net N$6: track 6.15 -> 0.06 mm

Commit message: Add files via upload
Parts:
- removed C3: 10uF, SparkFun-Capacitors:CPOL-RADIAL-100UF-25V
- removed C5: 470uF, SparkFun-Capacitors:CPOL-RADIAL-1000UF-25V
- removed D11, D7, D8, D9: 6V Zener, SparkFun-DiscreteSemi:DIODE-ZENER
- removed J11: (no value), SparkFun-Connectors:1X02
- removed LED1: (no value), adafruit:LED5MM
- removed R10: 330, resistor:0204/5
- removed R12: 46K, resistor:0204/5
- added C11, C12, C13: 330uF, SparkFun-Capacitors:CPOL-RADIAL-100UF-25V
- added J16: (no value), SparkFun-Connectors:1X08
- added JP1: JUMPER-PAD-2-NOYES_SILK, SparkFun-Passives:PAD-JUMPER-2-NO_YES_SILK
- added U$5, U$6: (no value), SparkFun-Electromechanical:STAND-OFF
- C4: value 100uF -> 330uF
- D3: value 1N4001 -> (none); device SparkFun-DiscreteSemi:DIODE-1N4001 -> adafruit:DO-1N4148
- J4: device SparkFun-Connectors:1X01 -> SparkFun-Connectors:1X05
- J8: device SparkFun-Connectors:1X04 -> SparkFun-Connectors:1X05
- J9: device SparkFun-Connectors:1X03 -> SparkFun-Connectors:1X05
- moved D1 126.1 mm to (61.0, 14.0)
- moved J2 118.9 mm to (26.7, 44.5), turned to 180 degrees
- moved J6 114.1 mm to (77.5, 31.8), turned to 180 degrees
- moved J5 113.2 mm to (77.5, 38.1), turned to 180 degrees
- moved D2 108.9 mm to (47.0, 12.7)
- moved C10 103.9 mm to (53.3, 20.3), turned to 90 degrees
- moved C9 101.2 mm to (61.0, 20.3), turned to 90 degrees
- moved J9 93.2 mm to (15.2, 3.81)
- moved J8 90.9 mm to (30.5, 3.81)
- moved C7 84.5 mm to (52.1, 34.3), turned to 180 degrees
- moved C1 77.3 mm to (52.1, 29.2), turned to 180 degrees
- moved Q2 68.3 mm to (45.7, 31.8), turned to 270 degrees
- moved C8 67.6 mm to (26.7, 27.9)
- moved C4 62.3 mm to (92.7, 29.2), turned to 270 degrees
- moved J1 56.2 mm to (76.2, 14.0), turned to 180 degrees
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Connections:
- removed net N$12: J3.7, U1.6
- removed net N$13: D2.C, J8.2
- removed net N$17: J3.10, U1.4
- removed net N$18: J8.1, J9.2
- removed net N$4 (its old number): C10.1, C6.2, C9.1, D1.C, J3.12, U1.20, U1.7
- removed net N$7: J8.3, U1.3
- removed net N$8: C5.+
- new net HWRXD: D2.C, J4.3
- new net HWTXD: J4.4, U1.3
- new net MISO: J2.1, U1.18
- new net MOSI: J2.4, U1.17
- new net N$20: D3.A, U1.25
- new net N$21: D3.C, J9.3
- new net N$22: J9.4, U1.26
- new net N$25: J8.3, U1.27
- new net N$26: J8.4, U1.28
- new net N$27: J16.1, J7.1
- new net N$28: J16.2, J7.2
- new net N$29: J16.3, J7.3
- new net N$30: J16.4, J7.4
- new net N$31: J16.5, J7.5
- new net N$32: J2.5, U1.1
- new net N$33: J16.6, J7.6
- new net N$34: J16.7, J7.7
- new net N$35: J16.8, J7.8
- new net SCK: J2.3, U1.19
- new net SS: U1.16
- new net VMCU: D1.A, J1.4
- net GND: now also C11.2, C12.2, C13.2, J2.6, J4.5, J8.5, J9.5; no longer C3.2, C5.-, D11.P$2, D7.P$2, D8.P$2, D9.P$2, J11.1, J8.4, LED1.K, R12.1
- net N$1: now also J3.7, U1.11; no longer LED1.A, R10.2
- net N$19: now also U1.24; no longer U1.28
- net N$5: now also J3.10, U1.6; no longer R12.2
- net VBAT: now also JP1.1
- net VBATSW: now also C13.1, C4.1
- net VCC: now also C10.1, C6.2, C9.1, D1.C, J2.2, J3.12, J4.2, J8.2, J9.2, U1.20, U1.7; no longer D1.A, J1.4, J9.1
- net VCEL: now also C11.1, C12.1, JP1.2
- net VSEN: now also J4.1, J8.1, J9.1; no longer J9.3
Routing:
- net VCC: track 0.00 -> 133.3 mm
- net VSEN: track 0.00 -> 84.3 mm
- net N$32: track 0.00 -> 52.5 mm
- net VBAT: track 0.00 -> 46.4 mm
- net VCEL: track 0.00 -> 46.4 mm
- net VBATSW: track 0.00 -> 40.6 mm
- net N$1: track 0.00 -> 40.4 mm
- net N$4: track 0.00 -> 40.2 mm
- net N$6: track 0.06 -> 38.3 mm
- net N$19: track 0.00 -> 37.4 mm
- net N$5: track 0.00 -> 37.3 mm
- net SCK: track 0.00 -> 32.1 mm
- net HWTXD: track 0.00 -> 24.7 mm
- net MISO: track 0.00 -> 21.2 mm
- net N$22: track 0.00 -> 19.6 mm
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Other:
- board text added: "Debug Console"
- board text added: "HW UART"
- board text added: "I2C"
- board text added: "Water Level Monitor V1 June 2017"
- board text removed: "10uF"
- board text removed: "470uF"
- board text removed: "AC Adapter"
- board text removed: "AC Adapter Relay"
- board text removed: "AtTiny84"
- board text removed: "Batt/Mains Status LED"
- board text removed: "Charge"
- board text removed: "Lighting UPS V4.1 May 2017"
- board text removed: "Mains Detect"
- board text removed: "Motion Det. enable"
- board text removed: "Motion Detect / Photocell"
- board text removed: "On/Off"
- board text removed: "Output to LED Lighting"
- board text removed: "P/B Mode"

Commit message: Add files via upload
Parts:
- added J10, J11: (no value), SparkFun-Connectors:1X01_NO_SILK
- added J12: (no value), SparkFun-Connectors:1X03_NO_SILK
- added J13, J14, J15: (no value), SparkFun-Connectors:1X02
- added J17: (no value), SparkFun-Connectors:2X4
- moved J16 13.4 mm to (16.5, 27.3)
- moved J7 13.3 mm to (3.81, 18.4)
- moved J2 7.75 mm to (22.2, 38.1), turned to 270 degrees
- moved U$1 2.54 mm to (7.62, 3.81)
- moved U$3 2.54 mm to (7.62, 45.7)
Connections:
- removed net SS: U1.16
- new net N$13: J10.1, J3.6
- new net N$37: J12.2, U1.13
- new net N$38: J12.3, U1.14
- new net N$5: J11.1, U1.4
- new net N$8: J12.1, U1.12
- new net SS1: J17.5, U1.16
- new net SS2: J17.7, U1.15
- net GND: now also J13.2, J14.2, J15.2, J17.6
- net MISO: now also J17.1
- net MOSI: now also J17.4
- net SCK: now also J17.3
- net VCC: now also J14.1, J17.2
- net VMCU: now also J15.1
- net VSEN: now also J13.1, J17.8
Routing:
- net SS2: track 0.00 -> 41.2 mm
- net SS1: track 0.00 -> 35.1 mm
- net VSEN: track 84.3 -> 115.7 mm
- net VCC: track 133.3 -> 161.4 mm
- net N$32: track 52.5 -> 34.1 mm
- net MISO: track 21.2 -> 34.6 mm
- net MOSI: track 10.7 -> 23.1 mm
- net SCK: track 32.1 -> 43.6 mm
- net N$5: track 0.00 -> 5.98 mm
- net VMCU: track 3.81 -> 8.89 mm
- net N$13: track 0.00 -> 2.79 mm
- net N$8: track 0.00 -> 2.54 mm
- net N$38: track 0.00 -> 2.54 mm
- net N$37: track 0.00 -> 2.54 mm
- net N$25: track 15.5 -> 18.1 mm
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Other:
- board text added: "+VCC"
- board text added: "+VMCU"
- board text added: "+VSEN"
- board text added: "330uF"
- board text added: "ISP"
- board text added: "MISO SCK SS1 SS2"
- board text added: "RI"
- board text added: "Rst"
- board text added: "SPI"
- board text added: "VCC MOSI GND VSEN"
- board text added: "VSEN VCC RX TX GND"
- board text added: "VSEN VCC SDA SCL GND"
- board text added: "Vio NS RX TX RI Key Rst SP- SP+ GND Bat"
- board text removed: "Shdn in gnd out"
- board text removed: "VCC"

Commit message: Add files via upload
Parts:
- removed C12, C13: 330uF, SparkFun-Capacitors:CPOL-RADIAL-100UF-25V
- removed D6: 16V Zener, SparkFun-DiscreteSemi:DIODE-ZENER
- removed Q4: 2N3904, SparkFun-DiscreteSemi:TO-92-AMMO
- removed R7: 10K, resistor:0204/5
- added C3: 0.1uF, SparkFun-Capacitors:CAP-PTH-SMALL
- added C5: 20pF, SparkFun-Capacitors:CAP-PTH-SMALL
- added D4: 16V Zener, SparkFun-DiscreteSemi:DIODE-ZENER
- added J18: (no value), SparkFun-Connectors:1X02
- added J19: (no value), SparkFun-Connectors:1X01_NO_SILK
- added J20, J22: (no value), SparkFun-Connectors:1X02_NO_SILK
- added LED1: (no value), led:LED5MM
- added Q3: NDP6020P, transistor-power:TO220BV
- added R2: 10K, resistor:0204/5
- added R4: 22K, resistor:0204/5
- C1: value 20pF -> 100uF; device SparkFun-Capacitors:CAP-PTH-SMALL -> SparkFun-Capacitors:CPOL-RADIAL-100UF-25V
- C10: value 100uF -> 330uF
- C2: value 0.01uF -> 100uF; device SparkFun-Passives:CAP-PTH-5MM -> SparkFun-Capacitors:CPOL-RADIAL-100UF-25V
- C4: value 330uF -> 20pF; device SparkFun-Capacitors:CPOL-RADIAL-100UF-25V -> SparkFun-Capacitors:CAP-PTH-SMALL
- C6: value 0.1uF -> 0.01uF; device SparkFun-Capacitors:CAP-PTH-SMALL -> SparkFun-Passives:CAP-PTH-5MM
- C7: value 20pF -> 330uF; device SparkFun-Capacitors:CAP-PTH-SMALL -> SparkFun-Capacitors:CPOL-RADIAL-100UF-25V
- C8: value 0.01uF -> 330uF; device SparkFun-Passives:CAP-PTH-5MM -> SparkFun-Capacitors:CPOL-RADIAL-100UF-25V
- C9: value 100uF -> 0.01uF; device SparkFun-Capacitors:CPOL-RADIAL-100UF-25V -> SparkFun-Passives:CAP-PTH-5MM
- J1: value D24V5F5 -> AVR_SPI_PRG_6PTH; device SparkFun-Connectors:1X04 -> SparkFun-Connectors:2X3
- J10: device SparkFun-Connectors:1X01_NO_SILK -> SparkFun-Connectors:1X12
- J11: device SparkFun-Connectors:1X01_NO_SILK -> SparkFun-Connectors:1X02
- J12: value (none) -> D24V5F5; device SparkFun-Connectors:1X03_NO_SILK -> SparkFun-Connectors:1X04
- J13: device SparkFun-Connectors:1X02 -> SparkFun-Connectors:1X03
- J14: device SparkFun-Connectors:1X02 -> SparkFun-Connectors:1X08
- J15: device SparkFun-Connectors:1X02 -> SparkFun-Connectors:2X4
- J16: value (none) -> D24V5F5; device SparkFun-Connectors:1X08 -> SparkFun-Connectors:1X04
- J17: value (none) -> RJ45; device SparkFun-Connectors:2X4 -> SparkFun-Connectors:RJ45-8
- J2: value AVR_SPI_PRG_6PTH -> (none); device SparkFun-Connectors:2X3 -> SparkFun-Connectors:1X02
- J3: device SparkFun-Connectors:1X12 -> SparkFun-Connectors:1X01_NO_SILK
- J4: device SparkFun-Connectors:1X05 -> SparkFun-Connectors:1X02_NO_SILK
- J5: value D24V5F5 -> (none); device SparkFun-Connectors:1X04 -> SparkFun-Connectors:1X01_NO_SILK
- J7: value RJ45 -> (none); device SparkFun-Connectors:RJ45-8 -> SparkFun-Connectors:1X04
- Q1: value NDP6020P -> (none); device transistor-power:TO220BV -> crystal:HC49U-V
- Q2: value (none) -> 2N3904; device crystal:HC49U-V -> SparkFun-DiscreteSemi:TO-92-AMMO
- R5: value 22K -> 10K
- R6: value 10K -> 330
- moved J2 75.1 mm to (91.4, 8.89), turned to 180 degrees
- moved C8 66.6 mm to (92.7, 36.8), turned to 90 degrees
- moved J15 64.3 mm to (9.53, 34.3), turned to 270 degrees
- moved J16 61.1 mm to (77.5, 31.8), turned to 180 degrees
- moved J1 59.1 mm to (22.2, 38.1), turned to 270 degrees
- moved J3 50.3 mm to (45.1, 18.4), turned to 0 degrees
- moved Q1 42.2 mm to (46.4, 31.8), turned to 270 degrees
- moved C10 40.4 mm to (92.7, 29.2), turned to 270 degrees
- moved J13 40.2 mm to (22.2, 19.7), turned to 90 degrees
- moved C4 40.0 mm to (52.7, 29.2), turned to 180 degrees
- moved J4 39.6 mm to (41.9, 43.2)
- moved J12 35.6 mm to (77.5, 38.1), turned to 180 degrees
- moved J14 33.5 mm to (16.5, 27.3), turned to 270 degrees
- moved C7 33.1 mm to (85.1, 36.8), turned to 90 degrees
- moved Q2 32.1 mm to (76.2, 21.6), turned to 90 degrees
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- renumbered X2 to X1
Connections:
- removed net N$37: J12.2, U1.13
- removed net N$38: J12.3, U1.14
- new net N$12: LED1.A, R6.1
- new net PB0: J4.1, U1.14
- new net PD6: J20.1, U1.12
- new net PD7: J22.1, U1.13
- net GND: now also C1.2, C3.1, C4.1, C5.1, C7.2, C8.2, D4.P$2, J1.6, J10.2, J11.2, J12.3, J15.6, J16.3, J18.2, J2.1, J20.2, J22.2, J4.2, J7.4, LED1.K, Q2.1, R5.1; no longer C1.1, C12.2, C13.2, C4.2, C7.1, C8.1, D6.P$2, J1.3, J14.2, J15.2, J17.6, J2.6, J3.2, J4.5, J5.3, Q4.1, R6.1
- net HWRXD: now also D3.C, J9.3; no longer D2.C, J4.3
- net HWTXD: now also J9.4; no longer J4.4
- net MISO: now also J1.1, J15.1; no longer J17.1, J2.1
- net MOSI: now also J1.4, J15.4; no longer J17.4, J2.4
- net N$1: now also J10.7; no longer J3.7
- net N$10: now also C5.2, Q1.1; no longer C7.2, Q2.1
- net N$11: now also C6.2; no longer C8.2
- net N$13: now also J10.6, J5.1; no longer J10.1, J3.6
- net N$14: now also Q2.3, R3.1; no longer Q4.3, R7.1
- net N$15: now also D3.A; no longer D2.A
- net N$19: now also R1.2; no longer R3.2
- net N$2: now also Q3.G, R2.1, R3.2; no longer Q1.G, R1.1, R7.2
- net N$20: now also D2.A; no longer D3.A
- net N$21: now also D2.C, J7.2; no longer D3.C, J9.3
- net N$22: now also J7.3; no longer J9.4
- net N$27: now also J14.1, J17.1; no longer J16.1, J7.1
- net N$28: now also J14.2, J17.2; no longer J16.2, J7.2
- net N$29: now also J14.3, J17.3; no longer J16.3, J7.3
- net N$3: now also Q2.2, R1.1; no longer Q4.2, R3.1
- net N$30: now also J14.4, J17.4; no longer J16.4, J7.4
- net N$31: now also J14.5, J17.5; no longer J16.5, J7.5
- net N$32: now also J1.5; no longer J2.5
- net N$33: now also J14.6, J17.6; no longer J16.6, J7.6
- net N$34: now also J14.7, J17.7; no longer J16.7, J7.7
- net N$35: now also J14.8, J17.8; no longer J16.8, J7.8
- net N$4: now also J10.9; no longer J3.9
- net N$5: now also J3.1; no longer J11.1
- net N$6: now also C9.1, R4.1, R5.2; no longer C2.1, R5.1, R6.2
- net N$7: now also J10.10; no longer J3.10
- net N$8: now also J19.1, R6.2; no longer J12.1, U1.12
- net N$9: now also C4.2, Q1.2; no longer C1.2, Q2.2
- net SCK: now also J1.3, J15.3; no longer J17.3, J2.3
- net SS1: now also J15.5; no longer J17.5
- net SS2: now also J15.7; no longer J17.7
- net VBAT: now also D4.P$1, J2.2, J6.2, Q3.S, R2.2; no longer D6.P$1, J1.2, Q1.S, R1.2
- net VBATSW: now also C10.1, C11.1, J12.2, J16.2, Q3.D, R4.2; no longer C13.1, C4.1, J5.2, J6.2, Q1.D, R5.2
- net VCC: now also D1.A, J1.2, J10.12, J11.1, J13.1, J15.2, J6.4, J7.1; no longer C10.1, C6.2, C9.1, D1.C, J14.1, J17.2, J2.2, J3.12, J4.2, U1.20, U1.7
- net VCEL: now also C7.1, C8.1, J10.1, J12.4; no longer C11.1, C12.1, J3.1, J5.4
- net VMCU: now also C1.1, C2.1, C3.2, D1.C, U1.20, U1.7; no longer D1.A, J1.4, J15.1
- net VSEN: now also J13.3, J15.8, J16.4, J18.1; no longer J13.1, J17.8, J4.1, J6.4
Routing:
- net VMCU: track 8.89 -> 40.7 mm
- net N$1: track 40.4 -> 51.3 mm
- net VBAT: track 46.4 -> 54.8 mm
- net VSEN: track 115.7 -> 123.5 mm
- net VBATSW: track 40.6 -> 38.0 mm
- net PD7: track 0.00 -> 2.54 mm
- net PD6: track 0.00 -> 2.54 mm
- net PB0: track 0.00 -> 2.54 mm
- net N$38: track 2.54 -> 0.00 mm
- net N$37: track 2.54 -> 0.00 mm
- net N$6: track 38.3 -> 40.8 mm
- net VCC: track 161.4 -> 159.0 mm
- net N$12: track 0.00 -> 1.91 mm
- net N$21: track 6.35 -> 5.08 mm
- net N$9: track 10.8 -> 11.3 mm
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Other:
- board text added: "+VBAT"
- board text added: "AtMega328P"
- board text added: "PB0 PD7 PD6"
- board text added: "PS"
- board text added: "VCC RX TX GND"
- board text added: "VSEN GND VCC"
- board text removed: "+VMCU"
- board text removed: "RI"

Commit message: Add files via upload
Parts:
- moved LED1 1.27 mm to (54.0, 45.7)
Routing:
- net N$12: track 1.91 -> 3.17 mm
Other:
- board text added: "PB0"
- board text added: "PD7 PD6"
- board text removed: "PB0 PD7 PD6"
Changed lines of the file:
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@@
 <text x="40.005" y="48.895" size="1.778" layer="21" rot="R180">Water Level Monitor
 V1 June 2017</text>
-<text x="80.01" y="25.4" size="1.27" layer="21" font="vector" rot="R180">2N3904</text>
+<text x="79.375" y="26.035" size="1.27" layer="21" font="vector" rot="R180">2N3904</text>
 <text x="83.185" y="22.86" size="1.27" layer="21" font="vector">NDP6020P</text>
 <text x="58.42" y="23.495" size="1.27" layer="21" font="vector">100uF</text>
@@
 GND
 VCC</text>
-<text x="50.165" y="37.465" size="1.3208" layer="21" font="vector" distance="90">PB0
-PD7
+<text x="50.165" y="37.465" size="1.3208" layer="21" font="vector" distance="90">PD7
 PD6</text>
 <text x="88.265" y="10.795" size="1.27" layer="21" font="vector" rot="R180" align="top-right">+VBAT</text>
+<text x="48.895" y="42.545" size="1.3208" layer="21" font="vector" distance="90">PB0</text>
 </plain>
 <attributes>
@@
 <attribute name="VALUE" x="70.7136" y="22.6314" size="0.9906" layer="27" ratio="10" rot="R180"/>
 </element>
-<element name="R4" library="resistor" package="0204/5" value="22K" x="69.85" y="27.94"/>
+<element name="R4" library="resistor" package="0204/5" value="22K" x="69.85" y="27.94" smashed="yes">
+<attribute name="NAME" x="69.1134" y="25.9334" size="0.9906" layer="25" ratio="10"/>
+<attribute name="VALUE" x="67.7164" y="25.6286" size="0.9906" layer="27" ratio="10"/>
+</element>
 <element name="R5" library="resistor" package="0204/5" value="10K" x="64.135" y="30.48" smashed="yes" rot="R270">
 <attribute name="NAME" x="65.3034" y="32.4866" size="0.9906" layer="25" ratio="10" rot="R270"/>
@@
 <attribute name="VALUE" x="49.1236" y="48.0314" size="0.9906" layer="27" ratio="10" rot="R180"/>
 </element>
-<element name="LED1" library="led" package="LED5MM" value="" x="52.705" y="45.72" smashed="yes">
-<attribute name="NAME" x="56.6166" y="43.815" size="1.27" layer="25" ratio="10" rot="R90"/>
-<attribute name="VALUE" x="55.9054" y="43.9166" size="1.27" layer="27" ratio="10"/>
+<element name="LED1" library="led" package="LED5MM" value="" x="53.975" y="45.72" smashed="yes">
+<attribute name="NAME" x="54.5084" y="44.45" size="1.27" layer="25" ratio="10" rot="R270"/>
+<attribute name="VALUE" x="57.1754" y="43.9166" size="1.27" layer="27" ratio="10"/>
 </element>
 <element name="J19" library="SparkFun-Connectors" package="1X01_NO_SILK" value="" x="41.91" y="45.72" smashed="yes">
@@
 <contactref element="U1" pad="1"/>
 <wire x1="39.37" y1="10.16" x2="38.1" y2="10.16" width="0.254" layer="1"/>
-<wire x1="38.1" y1="10.16" x2="34.29" y2="13.97" width="0.254" layer="1"/>
-<wire x1="34.29" y1="13.97" x2="34.29" y2="17.78" width="0.254" layer="1"/>
-<wire x1="34.29" y1="17.78" x2="33.02" y2="19.05" width="0.254" layer="1"/>
+<wire x1="38.1" y1="10.16" x2="35.56" y2="12.7" width="0.254" layer="1"/>
+<wire x1="35.56" y1="12.7" x2="35.56" y2="16.51" width="0.254" layer="1"/>
+<wire x1="35.56" y1="16.51" x2="33.02" y2="19.05" width="0.254" layer="1"/>
 <wire x1="22.225" y1="33.02" x2="22.225" y2="32.385" width="0.254" layer="1"/>
 <wire x1="22.225" y1="32.385" x2="24.13" y2="30.48" width="0.254" layer="1"/>
@@
 <contactref element="R6" pad="1"/>
 <contactref element="LED1" pad="A"/>
-<wire x1="49.53" y1="45.72" x2="51.435" y2="45.72" width="0.254" layer="1"/>
+<wire x1="49.53" y1="45.72" x2="52.705" y2="45.72" width="0.254" layer="1"/>
 </signal>
 </signals>
