File: hardware/WaterLevelMonitor_v1.brd (EAGLE design)
At the start: 98.7 x 49.5 mm, 55 parts, among them J1 AVR_SPI_PRG_6PTH, J12 D24V5F5, J16 D24V5F5, J17 RJ45, J21 POWER_JACKPTH_BREAD, J6 D24V5F5, Q2 2N3904, Q3 NDP6020P, U1 ATMEGA328P_PDIP

Commit message: Add files via upload
Parts:
- added J23: (no value), SparkFun-Connectors:1X01_NO_SILK
- moved D4 31.0 mm to (71.1, 4.45), turned to 180 degrees
Connections:
- new net N$16: J21.GNDBREAK, J23.1
Routing:
- net N$16: track 0.00 -> 4.62 mm
- net VBAT: track 80.4 -> 81.8 mm
Changed lines of the file:
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@@
 <element name="C10" library="SparkFun-Capacitors" package="CPOL-RADIAL-100UF-25V" value="330uF" x="92.71" y="29.21" rot="R270"/>
 <element name="C3" library="SparkFun-Capacitors" package="CAP-PTH-SMALL" value="0.1uF" x="48.26" y="18.415" rot="R90"/>
-<element name="D4" library="SparkFun-DiscreteSemi" package="DIODE-ZENER" value="16V Zener" x="96.52" y="22.225" rot="R90"/>
+<element name="D4" library="SparkFun-DiscreteSemi" package="DIODE-ZENER" value="16V Zener" x="71.12" y="4.445" rot="R180"/>
 <element name="J6" library="SparkFun-Connectors" package="1X04" value="D24V5F5" x="77.47" y="13.97" smashed="yes" rot="R180">
 <attribute name="PROD_ID" value="CONN-09696" x="77.47" y="13.97" size="1.778" layer="27" rot="R180" display="off"/>
@@
 <element name="J21" library="SparkFun-Connectors" package="POWER_JACK_PTH_BREAD" value="POWER_JACKPTH_BREAD" x="102.235" y="11.43" rot="R90">
 <attribute name="PROD_ID" value="PRT-10811" x="102.235" y="11.43" size="1.4224" layer="27" rot="R90" display="off"/>
+</element>
+<element name="J23" library="SparkFun-Connectors" package="1X01_NO_SILK" value="" x="95.25" y="18.415" smashed="yes">
+<attribute name="NAME" x="94.0562" y="16.4338" size="1.27" layer="25" rot="R90"/>
+<attribute name="VALUE" x="93.98" y="15.24" size="1.27" layer="27"/>
 </element>
 </elements>
@@
 <wire x1="74.93" y1="12.7" x2="74.93" y2="13.97" width="1.016" layer="16"/>
 <wire x1="80.01" y1="8.89" x2="80.01" y2="11.7" width="1.016" layer="16"/>
-<wire x1="96.52" y1="18.669" x2="90.424" y2="18.669" width="0.4064" layer="16"/>
 <wire x1="90.424" y1="18.669" x2="90.17" y2="18.415" width="0.4064" layer="16"/>
 <wire x1="90.17" y1="21.59" x2="90.17" y2="18.415" width="1.016" layer="1"/>
@@
 <wire x1="74.93" y1="12.7" x2="74.93" y2="13.97" width="1.016" layer="1"/>
 <wire x1="80.01" y1="8.89" x2="80.01" y2="11.43" width="1.016" layer="1"/>
+<wire x1="90.17" y1="21.844" x2="90.17" y2="21.59" width="0.4064" layer="16"/>
+<wire x1="74.676" y1="4.445" x2="75.565" y2="4.445" width="0.4064" layer="16"/>
+<wire x1="75.565" y1="4.445" x2="80.01" y2="8.89" width="0.4064" layer="16"/>
 </signal>
 <signal name="N$2">
@@
 <wire x1="49.53" y1="45.72" x2="52.705" y2="45.72" width="0.254" layer="1"/>
 </signal>
+<signal name="N$16">
+<contactref element="J21" pad="GNDBREAK"/>
+<contactref element="J23" pad="1"/>
+<wire x1="91.535" y1="16.23" x2="93.065" y2="16.23" width="0.4064" layer="16"/>
+<wire x1="93.065" y1="16.23" x2="95.25" y2="18.415" width="0.4064" layer="16"/>
+</signal>
 </signals>
